File: electronics/Sensor/Sensor.sch (KiCad schematic (older format))
At the start: 9 parts, among them J1 SS-60000-009, U1 OPA320AIDBVT

Commit message: split controller and sensor + add gerbers
Changed lines of the file:
@@
 $Descr A4 11693 8268
 encoding utf-8
-Sheet 1 2
+Sheet 1 1
 Title ""
 Date ""
@@
 $EndComp
 Connection ~ 4150 2150
-$Sheet
-S 4600 800  900  1000
-U 60497DFA
-F0 "TeensySide" 50
-F1 "TeensySide.sch" 50
-$EndSheet
 Text Label 3900 2350 3    50   ~ 0
 Fout
